Commit message: view_sensors.launch added

File: urdf/basic_sensors/gnss.urdf.xacro (robot description, xacro)
@@ -34,5 +34,5 @@
     <parent link="${parent}"/>
     <child link="${prefix}${index}_link"/>
-    <origin xyz="${x_loc} ${y_loc} ${z_loc}" rpy="0 0 0"/>
+    <xacro:insert_block name="origin"/>
   </joint>
   <gazebo reference="${prefix}${index}_link">

File: urdf/basic_sensors/imu.urdf.xacro (robot description, xacro)
@@ -29,5 +29,5 @@
     <parent link="${parent}"/>
     <child link="${prefix}_${name}_${index}_link"/>
-    <origin xyz="${x_loc} ${y_loc} ${z_loc}"/>
+    <xacro:insert_block name="origin"/>
   </joint>
   <gazebo reference="${prefix}_${name}_${index}_link">

File: urdf/basic_sensors/lidar2D.urdf.xacro (robot description, xacro)
@@ -34,6 +34,5 @@
     <parent link="${parent}"/>
     <child link="${prefix}_${name}_${index}_link"/>
-    <origin xyz="${x_loc} ${y_loc} ${z_loc}"/>
-    <!-- <origin xyz="0.215 0.0 0.30" rpy="0 0 0"/> -->
+     <xacro:insert_block name="origin"/>
   </joint>
   <gazebo reference="${prefix}_${name}_${index}_link">

File: urdf/load_all_sensors.urdf.xacro (robot description, xacro)
@@ -2,13 +2,14 @@
 <robot name="all_sensors" xmlns:xacro="http://wiki.ros.org/xacro">
      <!-- Include the BASIC SENSORS -->
-    <xacro:include filename="$(find robot_sim_sensors)/basic_sensors/monocamera.urdf.xacro" />
-    <xacro:include filename="$(find robot_sim_sensors)/basic_sensors/depthcam.urdf.xacro" />
-    <xacro:include filename="$(find robot_sim_sensors)/basic_sensors/wide_angle_camera.urdf.xacro" />
-    <xacro:include filename="$(find robot_sim_sensors)/basic_sensors/lidar2D.urdf.xacro" />
-    <xacro:include filename="$(find robot_sim_sensors)/basic_sensors/lidar3D.urdf.xacro" />
-    <xacro:include filename="$(find robot_sim_sensors)/basic_sensors/gnss.urdf.xacro" />
-    <xacro:include filename="$(find robot_sim_sensors)/basic_sensors/imu.urdf.xacro" />
-    <xacro:include filename="$(find robot_sim_sensors)/basic_sensors/bumper.urdf.xacro" />
+    <xacro:include filename="$(find robot_sim_sensors)/urdf/basic_sensors/monocamera.urdf.xacro" />
+    <xacro:include filename="$(find robot_sim_sensors)/urdf/basic_sensors/depthcam.urdf.xacro" />
+    <xacro:include filename="$(find robot_sim_sensors)/urdf/basic_sensors/wide_angle_camera.urdf.xacro" />
+    <xacro:include filename="$(find robot_sim_sensors)/urdf/basic_sensors/lidar2D.urdf.xacro" />
+    <xacro:include filename="$(find robot_sim_sensors)/urdf/basic_sensors/lidar3D.urdf.xacro" />
+    <xacro:include filename="$(find robot_sim_sensors)/urdf/basic_sensors/gnss.urdf.xacro" />
+    <xacro:include filename="$(find robot_sim_sensors)/urdf/basic_sensors/imu.urdf.xacro" />
+    <xacro:include filename="$(find robot_sim_sensors)/urdf/basic_sensors/bumper.urdf.xacro" />
     <!-- Include the BRAND SENSORS -->
-    <!-- <xacro:include filename="$(find robot_sim_sensors)/brand_sensors/..." /> -->
+    <!-- <xacro:include filename="$(find robot_sim_sensors)/urdf/brand_sensors/..." /> -->
+    <xacro:include filename="$(find robot_sim_sensors)/urdf/inertia.urdf.xacro" />
 </robot>

File: urdf/view_sensors.urdf.xacro (robot description, xacro)
@@ -1,8 +1,11 @@
 <?xml version="1.0"?>
 <robot name="view_sensors" xmlns:xacro="http://wiki.ros.org/xacro">
-    <!-- Flag to select the high or low quality model -->
+   <!-- Flag to select the high or low quality model -->
     <xacro:property name="hq" value="true" />
     <!-- <xacro:property name="robot_index" default="1" />-->
     <xacro:property name="prefix" default="robot_1" />
+    <xacro:include filename="$(find robot_sim_sensors)/urdf/load_all_sensors.urdf.xacro" />
+    <xacro:include filename="$(find robot_sim_sensors)/urdf/base_link.urdf.xacro" />
+    <xacro:base_link_sensors prefix="${prefix}" />
     <!-- ##################  BASIC SENSORS ################## -->
     <xacro:monocamera prefix="${prefix}" name="monocamera" index="front" parent="${prefix}_base_link" enabled="false" hq="${hq}" >
@@ -24,5 +27,5 @@
         <origin xyz="0.0 0.0 0.0" rpy="0 0 0"/>
     </xacro:imu_sensor>
-    <xacro:gnss prefix="${prefix}"  name="gnss"  parent="${prefix}_base_link" index="1" publish_bf="true"  enabled="false" hq="${hq}" >
+    <xacro:gnss prefix="${prefix}"  name="gnss"  parent="${prefix}_base_link" index="1"  enabled="false" hq="${hq}" >
         <origin xyz="0.0 0.0 0.0" rpy="0 0 0"/>
     </xacro:gnss>
