Commit message: change depthcam + change bumper

File: urdf/basic_sensors/bumper.urdf.xacro (robot description, xacro)
@@ -18,5 +18,5 @@
       </geometry>
     </visual>
-    <collision>
+    <collision name="bumper_collision">
       <geometry>
         <box size="0.1 0.1 0.1"/>
@@ -31,9 +31,14 @@
   </joint>
   <gazebo reference="${prefix}_${name}_${index}_link">
+    <material>Gazebo/Black</material>
+  </gazebo>
+  <gazebo reference="${prefix}_${name}_${index}_link">
     <gravity>true</gravity>
-        <sensor type="contact" name="${prefix}_${name}_${index}_link">
+    <max_contacts>1</max_contacts>
+        <sensor type="contact" name="${prefix}_${name}_${index}_sensor">
+          <always_on>true</always_on>
           <update_rate>60</update_rate>
           <contact>
-            <collision>collision</collision>
+            <collision>robot_base_link_fixed_joint_lump__bumper_collision_collision_2</collision>
           </contact>
           <plugin name="${prefix}_${name}_${index}_controller" filename="libgazebo_ros_bumper.so">
@@ -42,5 +47,5 @@
               <argument>bumper_states:=bumper</argument>
             </ros>
-            <frame_name>${prefix}_${name}_${index}_link</frame_name>
+            <frame_name>world</frame_name>
           </plugin>
         </sensor>

File: urdf/basic_sensors/depthcam.urdf.xacro (robot description, xacro)
@@ -14,34 +14,31 @@
       <link name="${prefix}_${name}_${index}_link">
         <visual>
-          <geometry>
-            <box size="0.01 0.01 0.01"/>
-          </geometry>
-          <origin rpy=" 1.57 0 1.57" xyz="0 0 0.0" />
+          <origin xyz="-0.05 0 0" rpy="0 0 1.57"/>
+            <geometry>
+              <box size="0.001 0.001 0.001"/>
+            </geometry>
         </visual>
-      <collision>
-        <geometry>
-          <origin rpy=" 1.57 0 1.57" xyz="0 0 0.0" />
-        </geometry>
-      </collision>
-      <xacro:box_inertia m="0.01" w="0.01" d="0.01" h="0.01"/>
+        <collision>
+          <origin xyz="-0.05 0 0" rpy="0 0 1.57"/>
+            <geometry>
+              <box size="0.001 0.001 0.001" />
+            </geometry>
+        </collision>
+        <xacro:box_inertia m="0.000001" w="0.001" d="0.001" h="0.001"/>
       </link>
       <link name="${prefix}_${name}_${index}_link_depthcloud">
         <visual>
           <geometry>
-              <box size="0.01 0.01 0.01" />
+              <box size="0.001 0.001 0.001" />
           </geometry>
-          <origin rpy="0 0 0" xyz="0 0 0.0" />
-      </visual>
-      <inertial>
-          <mass value="0.03" />
-          <origin xyz="0 0 0" rpy="0 0 0" />
-          <inertia ixx="0.0006" ixy="0.00" ixz="0" iyy="0.0005" iyz="0" izz="0.0007"/>
-      </inertial>
-      <collision>
+            <origin rpy="0 0 0" xyz="0 0 0"/>
+        </visual>
+        <xacro:box_inertia m="0.000001" w="0.001" d="0.001" h="0.001"/>
+        <collision>
           <geometry>
-              <box size="0.01 0.01 0.01" />
+              <box size="0.001 0.001 0.001"/>
           </geometry>
-          <origin rpy="0 0 0" xyz="0 0 0.0" />
-      </collision>
+          <origin rpy="0 0 0" xyz="0 0 0"/>
+        </collision>
       </link>
       <joint name="${prefix}_${name}_${index}_joint" type="fixed">
@@ -51,7 +48,7 @@
       </joint>
       <joint name="${prefix}_${name}_${index}_joint_pointcloud" type="fixed">
-          <parent link="${prefix}_${name}_${index}_link" />
-          <child link="${prefix}_${name}_${index}_link_depthcloud" />
-          <origin xyz="0 0 0" rpy="-1.57 0 -1.57"  />
+          <parent link="${prefix}_${name}_${index}_link"/>
+          <child link="${prefix}_${name}_${index}_link_depthcloud"/>
+          <origin xyz="0 0 0" rpy="-1.57 0 -1.57" />
       </joint>
       <gazebo reference="${prefix}_${name}_${index}_link">

Commit message: change ${prefix}_ to ${prefix} in all frame and joints

File: urdf/basic_sensors/bumper.urdf.xacro (robot description, xacro)
@@ -12,5 +12,5 @@
   <!-- *********************** IMU SETUP *********************************  -->
   <!-- Each sensor must be attached to a link.                              -->
-  <link name="${prefix}_${name}_${index}_link">
+  <link name="${prefix}${name}_${index}_link">
     <visual>
       <geometry>
@@ -25,16 +25,16 @@
     <xacro:box_inertia m="0.1" w="0.1" d="0.1" h="0.1"/>
   </link>
-  <joint name="${prefix}_${name}_${index}_joint" type="fixed">
+  <joint name="${prefix}${name}_${index}_joint" type="fixed">
     <parent link="${parent}"/>
-    <child link="${prefix}_${name}_${index}_link"/>
+    <child link="${prefix}${name}_${index}_link"/>
     <xacro:insert_block name="origin"/>
   </joint>
-  <gazebo reference="${prefix}_${name}_${index}_link">
+  <gazebo reference="${prefix}${name}_${index}_link">
     <material>Gazebo/Black</material>
   </gazebo>
-  <gazebo reference="${prefix}_${name}_${index}_link">
+  <gazebo reference="${prefix}${name}_${index}_link">
     <gravity>true</gravity>
     <max_contacts>1</max_contacts>
-        <sensor type="contact" name="${prefix}_${name}_${index}_sensor">
+        <sensor type="contact" name="${prefix}${name}_${index}_sensor">
           <always_on>true</always_on>
           <update_rate>60</update_rate>
@@ -42,5 +42,5 @@
             <collision>robot_base_link_fixed_joint_lump__bumper_collision_collision_2</collision>
           </contact>
-          <plugin name="${prefix}_${name}_${index}_controller" filename="libgazebo_ros_bumper.so">
+          <plugin name="${prefix}${name}_${index}_controller" filename="libgazebo_ros_bumper.so">
             <ros>
               <namespace>${prefix}</namespace>

File: urdf/basic_sensors/depthcam.urdf.xacro (robot description, xacro)
@@ -12,5 +12,5 @@
     <!-- *********************** DEPTHCAM SETUP *********************************  -->
     <!-- Each sensor must be attached to a link.                              -->
-      <link name="${prefix}_${name}_${index}_link">
+      <link name="${prefix}${name}_${index}_link">
         <visual>
           <origin xyz="-0.05 0 0" rpy="0 0 1.57"/>
@@ -27,5 +27,5 @@
         <xacro:box_inertia m="0.000001" w="0.001" d="0.001" h="0.001"/>
       </link>
-      <link name="${prefix}_${name}_${index}_link_depthcloud">
+      <link name="${prefix}${name}_${index}_link_depthcloud">
         <visual>
           <geometry>
@@ -42,15 +42,15 @@
         </collision>
       </link>
-      <joint name="${prefix}_${name}_${index}_joint" type="fixed">
+      <joint name="${prefix}${name}_${index}_joint" type="fixed">
         <parent link="${parent}"/>
-        <child link="${prefix}_${name}_${index}_link"/>
+        <child link="${prefix}${name}_${index}_link"/>
         <xacro:insert_block name="origin"/>
       </joint>
-      <joint name="${prefix}_${name}_${index}_joint_pointcloud" type="fixed">
+      <joint name="${prefix}${name}_${index}_joint_pointcloud" type="fixed">
           <parent link="${prefix}_${name}_${index}_link"/>
           <child link="${prefix}_${name}_${index}_link_depthcloud"/>
           <origin xyz="0 0 0" rpy="-1.57 0 -1.57" />
       </joint>
-      <gazebo reference="${prefix}_${name}_${index}_link">
+      <gazebo reference="${prefix}${name}_${index}_link">
         <gravity>true</gravity>
         <sensor name="${name}_${index}" type="depth">
@@ -79,5 +79,5 @@
                 </noise>
               </camera>
-          <plugin name="${prefix}_${name}_${index}_controller" filename="libgazebo_ros_camera.so">
+          <plugin name="${prefix}${name}_${index}_controller" filename="libgazebo_ros_camera.so">
                 <ros>
                   <namespace>${prefix}</namespace>
@@ -95,5 +95,5 @@
                 <min_depth>0.1</min_depth>
                 <max_depth>500</max_depth>
-                <frame_name>${prefix}_${name}_${index}_link_depthcloud</frame_name>
+                <frame_name>${prefix}${name}_${index}_link_depthcloud</frame_name>
           </plugin>
         </sensor>

File: urdf/basic_sensors/imu.urdf.xacro (robot description, xacro)
@@ -13,5 +13,5 @@
   <!-- *********************** IMU SETUP *********************************  -->
   <!-- Each sensor must be attached to a link.                              -->
-  <link name="${prefix}_${name}_${index}_link">
+  <link name="${prefix}${name}_${index}_link">
     <visual>
       <geometry>
@@ -26,12 +26,12 @@
     <xacro:box_inertia m="0.1" w="0.1" d="0.1" h="0.1"/>
   </link>
-  <joint name="${prefix}_${name}_${index}_joint" type="fixed">
+  <joint name="${prefix}${name}_${index}_joint" type="fixed">
     <parent link="${parent}"/>
-    <child link="${prefix}_${name}_${index}_link"/>
+    <child link="${prefix}${name}_${index}_link"/>
     <xacro:insert_block name="origin"/>
   </joint>
-  <gazebo reference="${prefix}_${name}_${index}_link">
+  <gazebo reference="${prefix}${name}_${index}_link">
     <gravity>true</gravity>
-    <sensor name="${prefix}_${name}_${index}" type="imu">
+    <sensor name="${prefix}${name}_${index}" type="imu">
       <always_on>true</always_on>
       <update_rate>100</update_rate>
@@ -111,7 +111,7 @@
         </linear_acceleration>
       </imu>
-      <plugin name="${prefix}_${name}_${index}_controller" filename="libgazebo_ros_imu_sensor.so">
+      <plugin name="${prefix}${name}_${index}_controller" filename="libgazebo_ros_imu_sensor.so">
         <initial_orientation_as_reference>false</initial_orientation_as_reference>
-        <frame_name>${prefix}_${name}_${index}_link</frame_name>
+        <frame_name>${prefix}${name}_${index}_link</frame_name>
         <ros>
           <namespace>/imu</namespace>

File: urdf/basic_sensors/lidar2D.urdf.xacro (robot description, xacro)
@@ -12,5 +12,5 @@
       <xacro:if value="${enabled}">
   <!-- *********************** LIDAR SETUP **********************************  -->
- <link name="${prefix}_${name}_${index}_link">
+ <link name="${prefix}${name}_${index}_link">
     <inertial>
       <origin xyz="0 0 0" rpy="0 0 0"/>
@@ -31,11 +31,11 @@
     </visual>
   </link>
-  <joint name="${prefix}_${name}_${index}_joint" type="fixed">
+  <joint name="${prefix}${name}_${index}_joint" type="fixed">
     <parent link="${parent}"/>
-    <child link="${prefix}_${name}_${index}_link"/>
+    <child link="${prefix}${name}_${index}_link"/>
      <xacro:insert_block name="origin"/>
   </joint>
-  <gazebo reference="${prefix}_${name}_${index}_link">
-    <sensor name="{name}_${index}" type="ray">
+  <gazebo reference="${prefix}${name}_${index}_link">
+    <sensor name="${prefix}${name}_${index}" type="ray">
       <always_on>true</always_on>
       <visualize>false</visualize>
@@ -61,5 +61,5 @@
         </noise>
       </ray>
-      <plugin name="${prefix}_${name}_${index}_controller" filename="libgazebo_ros_ray_sensor.so">
+      <plugin name="${prefix}${name}_${index}_controller" filename="libgazebo_ros_ray_sensor.so">
         <ros>
           <namespace>${prefix}</namespace>
@@ -67,5 +67,5 @@
         </ros>
         <output_type>sensor_msgs/LaserScan</output_type>
-        <frame_name>${prefix}_${name}_${index}_link</frame_name>
+        <frame_name>${prefix}${name}_${index}_link</frame_name>
       </plugin>
     </sensor>

File: urdf/basic_sensors/lidar3D.urdf.xacro (robot description, xacro)
@@ -12,5 +12,5 @@
       <xacro:if value="${enabled}">
   <!-- *********************** LIDAR SETUP **********************************  -->
- <link name="${prefix}_${name}_${index}_link">
+ <link name="${prefix}${name}_${index}_link">
     <inertial>
       <origin xyz="0 0 0" rpy="0 0 0"/>
@@ -31,11 +31,11 @@
     </visual>
   </link>
-  <joint name="${prefix}_${name}_${index}_joint" type="fixed">
+  <joint name="${prefix}${name}_${index}_joint" type="fixed">
     <parent link="${parent}"/>
-    <child link="${prefix}_${name}_${index}_link"/>
+    <child link="${prefix}${name}_${index}_link"/>
     <xacro:insert_block name="origin"/>
   </joint>
-  <gazebo reference="${prefix}_${name}_${index}_link">
-    <sensor name="${name}_${index}" type="gpu_ray">
+  <gazebo reference="${prefix}${name}_${index}_link">
+    <sensor name="${prefix}${name}_${index}" type="gpu_ray">
       <always_on>true</always_on>
       <visualize>true</visualize>
@@ -67,5 +67,5 @@
         </noise>
       </ray>
-      <plugin name="${prefix}_${name}_${index}_controller" filename="libgazebo_ros_ray_sensor.so">
+      <plugin name="${prefix}${name}_${index}_controller" filename="libgazebo_ros_ray_sensor.so">
         <ros>
           <namespace>${prefix}</namespace>
@@ -73,5 +73,5 @@
         </ros>
         <output_type>sensor_msgs/PointCloud2</output_type>
-        <frame_name>${prefix}_${name}_${index}_link</frame_name>
+        <frame_name>${prefix}${name}_${index}_link</frame_name>
       </plugin>
     </sensor>

File: urdf/basic_sensors/monocamera.urdf.xacro (robot description, xacro)
@@ -26,12 +26,12 @@
      <xacro:box_inertia m="0.1" w="0.1" d="0.1" h="0.1"/>
   </link>
-  <joint name="${prefix}_${name}_${index}_joint" type="fixed">
+  <joint name="${prefix}${name}_${index}_joint" type="fixed">
     <parent link="${parent}"/>
-    <child link="${prefix}_${name}_${index}_link"/>
+    <child link="${prefix}${name}_${index}_link"/>
     <xacro:insert_block name="origin"/>
   </joint>
-  <gazebo reference="${prefix}_${name}_${index}_link">
+  <gazebo reference="${prefix}${name}_${index}_link">
     <gravity>true</gravity>
-    <sensor name="${name}_${index}" type="camera">
+    <sensor name="${prefix}${name}_${index}" type="camera">
        <update_rate>30</update_rate>
           <visualize>false</visualize>
@@ -56,5 +56,5 @@
             </noise>
           </camera>
-      <plugin name="${prefix}_${name}_${index}_controller" filename="libgazebo_ros_camera.so">
+      <plugin name="${prefix}${name}_${index}_controller" filename="libgazebo_ros_camera.so">
             <ros>
              <namespace>${prefix}</namespace>

File: urdf/basic_sensors/stereocam.urdf.xacro (robot description, xacro)
@@ -26,12 +26,12 @@
       <xacro:box_inertia m="0.1" w="0.1" d="0.1" h="0.1"/>
       </link>
-      <joint name="${prefix}_${name}_${index}_joint" type="fixed">
+      <joint name="${prefix}${name}_${index}_joint" type="fixed">
         <parent link="${parent}"/>
-        <child link="${prefix}_${name}_${index}_link"/>
+        <child link="${prefix}${name}_${index}_link"/>
         <xacro:insert_block name="origin"/>
       </joint>
-      <gazebo reference="${prefix}_${name}_${index}_link">
+      <gazebo reference="${prefix}${name}_${index}_link">
         <gravity>true</gravity>
-        <sensor name="${name}_${index}" type="multicamera">
+        <sensor name="${prefix}${name}_${index}" type="multicamera">
           <update_rate>60</update_rate>
               <visualize>false</visualize>
@@ -79,5 +79,5 @@
             </noise>
           </camera>
-          <plugin name="${prefix}_${name}_${index}_controller" filename="libgazebo_ros_camera.so">
+          <plugin name="${prefix}${name}_${index}_controller" filename="libgazebo_ros_camera.so">
                 <ros>
                   <namespace>${prefix}</namespace>

File: urdf/basic_sensors/wide_angle_camera.urdf.xacro (robot description, xacro)
@@ -11,5 +11,5 @@
   <xacro:macro name="wide_angle_camera" params="prefix:='' name:='' index parent *origin enabled hq">
     <xacro:if value="${enabled}">                           -->
-    <link name="${prefix}_${name}_${index}_link">
+    <link name="${prefix}${name}_${index}_link">
     <visual>
      <geometry>
@@ -24,12 +24,12 @@
      <xacro:box_inertia m="0.1" w="0.1" d="0.1" h="0.1"/>
   </link>
-  <joint name="${prefix}_${name}_${index}_joint" type="fixed">
+  <joint name="${prefix}${name}_${index}_joint" type="fixed">
     <parent link="${parent}"/>
-    <child link="${prefix}_${name}_${index}_link"/>
+    <child link="${prefix}${name}_${index}_link"/>
     <xacro:insert_block name="origin"/>
   </joint>
-  <gazebo reference="${prefix}_${name}_${index}_link">
+  <gazebo reference="${prefix}${name}_${index}_link">
     <gravity>true</gravity>
-    <sensor name="${name}_${index}" type="wideanglecamera">
+    <sensor name="${prefix}${name}_${index}" type="wideanglecamera">
     <camera>
        <horizontal_fov>6.283</horizontal_fov>
@@ -69,5 +69,5 @@
     <update_rate>30</update_rate>
     </camera>
-      <plugin name="${prefix}_${name}_${index}_controller" filename="libgazebo_ros_camera.so">
+      <plugin name="${prefix}${name}_${index}_controller" filename="libgazebo_ros_camera.so">
             <ros>
              <namespace>${prefix}</namespace>

File: urdf/brand_sensors/zed2i.urdf.xacro (robot description, xacro)
@@ -12,5 +12,5 @@
     <!-- *********************** DEPTHCAM SETUP *********************************  -->
     <!-- Each sensor must be attached to a link.                              -->
-      <link name="${prefix}_${name}_${index}_link">
+      <link name="${prefix}${name}_${index}_link">
         <visual>
           <origin rpy=" 0 0 1.57" xyz="-0.05 0 0.0" />
@@ -29,5 +29,5 @@
       <xacro:box_inertia m="0.01" w="0.01" d="0.01" h="0.01"/>
       </link>
-      <link name="${prefix}_${name}_${index}_link_depthcloud">
+      <link name="${prefix}${name}_${index}_link_depthcloud">
         <visual>
           <geometry>
@@ -48,17 +48,17 @@
       </collision>
       </link>
-      <joint name="${prefix}_${name}_${index}_joint" type="fixed">
+      <joint name="${prefix}${name}_${index}_joint" type="fixed">
         <parent link="${parent}"/>
-        <child link="${prefix}_${name}_${index}_link"/>
+        <child link="${prefix}${name}_${index}_link"/>
         <xacro:insert_block name="origin"/>
       </joint>
-      <joint name="${prefix}_${name}_${index}_joint_pointcloud" type="fixed">
-          <parent link="${prefix}_${name}_${index}_link" />
-          <child link="${prefix}_${name}_${index}_link_depthcloud" />
+      <joint name="${prefix}${name}_${index}_joint_pointcloud" type="fixed">
+          <parent link="${prefix}${name}_${index}_link" />
+          <child link="${prefix}${name}_${index}_link_depthcloud" />
           <origin xyz="0.0 0.0 0.0" rpy="-1.57 0 -1.57"  />
       </joint>
-      <gazebo reference="${prefix}_${name}_${index}_link">
+      <gazebo reference="${prefix}${name}_${index}_link">
         <gravity>true</gravity>
-        <sensor name="${name}_${index}" type="depth">
+        <sensor name="${prefix}${name}_${index}" type="depth">
           <update_rate>60</update_rate>
               <visualize>false</visualize>
@@ -85,5 +85,5 @@
                 </noise>
               </camera>
-          <plugin name="${prefix}_${name}_${index}_controller" filename="libgazebo_ros_camera.so">
+          <plugin name="${prefix}${name}_${index}_controller" filename="libgazebo_ros_camera.so">
                 <ros>
                   <namespace>${prefix}</namespace>
@@ -101,5 +101,5 @@
                 <min_depth>0.1</min_depth>
                 <max_depth>500</max_depth>
-                <frame_name>${prefix}_${name}_${index}_link_depthcloud</frame_name>
+                <frame_name>${prefix}${name}_${index}_link_depthcloud</frame_name>
           </plugin>
         </sensor>
