Commit message: change prefix_ to prefix

File: urdf/basic_sensors/depthcam.urdf.xacro (robot description, xacro)
@@ -48,11 +48,11 @@
       </joint>
       <joint name="${prefix}${name}_${index}_joint_pointcloud" type="fixed">
-          <parent link="${prefix}_${name}_${index}_link"/>
-          <child link="${prefix}_${name}_${index}_link_depthcloud"/>
+          <parent link="${prefix}${name}_${index}_link"/>
+          <child link="${prefix}${name}_${index}_link_depthcloud"/>
           <origin xyz="0 0 0" rpy="-1.57 0 -1.57" />
       </joint>
       <gazebo reference="${prefix}${name}_${index}_link">
         <gravity>true</gravity>
-        <sensor name="${name}_${index}" type="depth">
+        <sensor name="${prefix}${name}_${index}" type="depth">
           <update_rate>60</update_rate>
               <visualize>false</visualize>

File: urdf/basic_sensors/gnss.urdf.xacro (robot description, xacro)
@@ -12,5 +12,5 @@
       <xacro:if value="${enabled}">
   <!-- *********************** LIDAR SETUP **********************************  -->
- <link name="${prefix}${index}_link">
+ <link name="${prefix}${name}_${index}_link">
     <inertial>
       <origin xyz="0 0 0" rpy="0 0 0"/>
@@ -31,11 +31,11 @@
     </visual>
   </link>
-  <joint name="${prefix}${index}_joint" type="fixed">
+  <joint name="${prefix}${name}_${index}_joint" type="fixed">
     <parent link="${parent}"/>
-    <child link="${prefix}${index}_link"/>
+    <child link="${prefix}${name}_${index}_link"/>
     <xacro:insert_block name="origin"/>
   </joint>
-  <gazebo reference="${prefix}${index}_link">
-      <sensor name="${prefix}${index}" type="gps">
+  <gazebo reference="${prefix}${name}_${index}_link">
+      <sensor name="${prefix}${name}_${index}" type="gps">
           <always_on>true</always_on>
           <update_rate>30</update_rate>
@@ -56,5 +56,5 @@
             </position_sensing>
           </gps>
-          <plugin name="${prefix}${index}_controller" filename="libgazebo_ros_gps_sensor.so">
+          <plugin name="${prefix}${name}_${index}_controller" filename="libgazebo_ros_gps_sensor.so">
             <ros>
               <namespace>/gps</namespace>
