Commit message: Add stereocam

File: urdf/load_all_sensors.urdf.xacro (robot description, xacro)
@@ -5,4 +5,5 @@
     <xacro:include filename="$(find robot_sim_sensors)/urdf/basic_sensors/depthcam.urdf.xacro" />
     <xacro:include filename="$(find robot_sim_sensors)/urdf/basic_sensors/wide_angle_camera.urdf.xacro" />
+    <xacro:include filename="$(find robot_sim_sensors)/urdf/basic_sensors/stereocam.urdf.xacro" />
     <xacro:include filename="$(find robot_sim_sensors)/urdf/basic_sensors/lidar2D.urdf.xacro" />
     <xacro:include filename="$(find robot_sim_sensors)/urdf/basic_sensors/lidar3D.urdf.xacro" />

File: urdf/view_sensors.urdf.xacro (robot description, xacro)
@@ -18,8 +18,11 @@
         <origin xyz="0.3 0.05 0.23" rpy="0 0 0"/>
     </xacro:depthcam>
+    <xacro:stereocam prefix="${prefix}" name="stereocam" index="1" parent="${prefix}_base_link"  enabled="true" hq="${hq}">
+        <origin xyz="0.3 0.05 0.23" rpy="0 0 0"/>
+    </xacro:stereocam>
     <xacro:lidar2D prefix="${prefix}" name="lidar2D" index="1" parent="${prefix}_base_link"   enabled="false" hq="${hq}">
         <origin xyz="0.3 -0.05 0.23" rpy="0 0 0"/>
     </xacro:lidar2D>
-    <xacro:lidar3D prefix="${prefix}" name="lidar3D" index="1" parent="${prefix}_base_link" enabled="true" hq="${hq}">
+    <xacro:lidar3D prefix="${prefix}" name="lidar3D" index="1" parent="${prefix}_base_link" enabled="false" hq="${hq}">
         <origin xyz="0.20 0.0 0.30" rpy="0 0 0"/>
     </xacro:lidar3D>
