Commit message: Add Zed2I to view_sensors file

File: urdf/view_sensors.urdf.xacro (robot description, xacro)
@@ -33,3 +33,6 @@
         <origin xyz="0.0 0.0 0.0" rpy="0 0 0"/>
     </xacro:gnss>
+    <xacro:zed2i prefix="${prefix}" name="depthcam" parent="${prefix}_base_link" index="1"  hq="${hq}" enabled="true">
+                <origin xyz="0.3 0.0 0.0" rpy="0 0 0"/>
+    </xacro:zed2i>
 </robot>
