Commit message: Add brand sensor zed2i

File: urdf/brand_sensors/zed2i.urdf.xacro (robot description, xacro)
@@ -8,5 +8,5 @@
     </inertial>
   </xacro:macro>
-  <xacro:macro name="depthcam" params="prefix:='' name:='' index parent *origin enabled hq">
+  <xacro:macro name="zed2i" params="prefix:='' name:='' index parent *origin enabled hq">
     <xacro:if value="${enabled}">
     <!-- *********************** DEPTHCAM SETUP *********************************  -->
@@ -14,12 +14,15 @@
       <link name="${prefix}_${name}_${index}_link">
         <visual>
+          <origin rpy=" 0 0 1.57" xyz="0 0 0.0" />
           <geometry>
-            <box size="0.01 0.01 0.01"/>
+            <!-- <box size="0.01 0.01 0.01"/> -->
+            <mesh scale="0.001 0.001 0.001" filename="file://$(find robot_sim_sensors)/urdf/brand_sensors/meshes/ZED2i.stl" />
           </geometry>
-          <origin rpy=" 1.57 0 1.57" xyz="0 0 0.0" />
         </visual>
       <collision>
+        <origin rpy=" 0 0 1.57" xyz="0 0 0.0" />
         <geometry>
-          <origin rpy=" 1.57 0 1.57" xyz="0 0 0.0" />
+          <!-- <mesh scale="0.001 0.001 0.001" filename="file://$(find robot_sim_sensors)/urdf/brand_sensors/meshes/ZED2i.stl" /> -->
+          <box size="0.001 0.001 0.001" />
         </geometry>
       </collision>
@@ -40,5 +43,5 @@
       <collision>
           <geometry>
-              <box size="0.01 0.01 0.01" />
+              <box size="0.001 0.001 0.001" />
           </geometry>
           <origin rpy="0 0 0" xyz="0 0 0.0" />
@@ -53,5 +56,5 @@
           <parent link="${prefix}_${name}_${index}_link" />
           <child link="${prefix}_${name}_${index}_link_depthcloud" />
-          <origin xyz="0 0 0" rpy="-1.57 0 -1.57"  />
+          <origin xyz="0.1 0 0" rpy="-1.57 0 -1.57"  />
       </joint>
       <gazebo reference="${prefix}_${name}_${index}_link">

File: urdf/load_all_sensors.urdf.xacro (robot description, xacro)
@@ -12,5 +12,5 @@
     <xacro:include filename="$(find robot_sim_sensors)/urdf/basic_sensors/bumper.urdf.xacro" />
     <!-- Include the BRAND SENSORS -->
-    <!-- <xacro:include filename="$(find robot_sim_sensors)/urdf/brand_sensors/..." /> -->
+    <xacro:include filename="$(find robot_sim_sensors)/urdf/brand_sensors/zed2i.urdf.xacro" />
     <xacro:include filename="$(find robot_sim_sensors)/urdf/inertia.urdf.xacro" />
 </robot>

Commit message: change orientation of sensor

File: urdf/brand_sensors/zed2i.urdf.xacro (robot description, xacro)
@@ -14,5 +14,5 @@
       <link name="${prefix}_${name}_${index}_link">
         <visual>
-          <origin rpy=" 0 0 1.57" xyz="0 0 0.0" />
+          <origin rpy=" 0 0 1.57" xyz="-0.05 0 0.0" />
           <geometry>
             <!-- <box size="0.01 0.01 0.01"/> -->
@@ -21,5 +21,5 @@
         </visual>
       <collision>
-        <origin rpy=" 0 0 1.57" xyz="0 0 0.0" />
+        <origin rpy=" 0 0 1.57" xyz="-0.05 0 0.0" />
         <geometry>
           <!-- <mesh scale="0.001 0.001 0.001" filename="file://$(find robot_sim_sensors)/urdf/brand_sensors/meshes/ZED2i.stl" /> -->
@@ -56,5 +56,5 @@
           <parent link="${prefix}_${name}_${index}_link" />
           <child link="${prefix}_${name}_${index}_link_depthcloud" />
-          <origin xyz="0.1 0 0" rpy="-1.57 0 -1.57"  />
+          <origin xyz="0.0 0.0 0.0" rpy="-1.57 0 -1.57"  />
       </joint>
       <gazebo reference="${prefix}_${name}_${index}_link">
@@ -74,5 +74,5 @@
                 <clip>
                   <near>0.02</near>
-                  <far>300</far>
+                  <far>20</far>
                 </clip>
                 <noise>

Commit message: change color of zed2i

File: urdf/brand_sensors/zed2i.urdf.xacro (robot description, xacro)
@@ -59,4 +59,10 @@
       </joint>
       <gazebo reference="${prefix}${name}_${index}_link">
+        <material>Gazebo/Black</material>
+      </gazebo>
+      <gazebo reference="${prefix}${name}_${index}_link_depthcloud">
+        <material>Gazebo/Black</material>
+      </gazebo>
+      <gazebo reference="${prefix}${name}_${index}_link">
         <gravity>true</gravity>
         <sensor name="${prefix}${name}_${index}" type="depth">
